File: projects/HA_control_SSRs/HA_control_SSRs.kicad_pcb (KiCad board)
At the start: 0 parts

Commit message: snapshot
Parts:
- added D1: IR26-21C_L110_TR8, LED_SMD:LED_1206_3216Metric, F.Cu at (134.8, 57.1)
- added Q1: MMBT3904, Package_TO_SOT_SMD:SOT-23, F.Cu at (108.0, 69.8)
- added R1: 1k, Resistor_SMD:R_1206_3216Metric_Pad1.30x1.75mm_HandSolder, F.Cu at (95.2, 69.8)
- added R2: 1k, Resistor_SMD:R_1206_3216Metric_Pad1.30x1.75mm_HandSolder, F.Cu at (127.0, 57.1)
- added U1: MCP23017M, UH_HA:Module_MCP23017, F.Cu at (76.2, 76.2)
- added U2: ASSR-1218, Package_SO:SO-4_4.4x4.3mm_P2.54mm, F.Cu at (120.7, 63.5)
Routing:
- added copper zone on F.Cu, net GND
Other:
- copper layers 0 -> 2
