File: projects/HA_control_SSRs/HA_control_SSRs.kicad_sch (KiCad schematic)
At the start: 3 parts, among them Q1 2N3904, U1 MCP23017M, U2 ASSR-1218

Commit message: snapshot
Parts:
- removed Q1: 2N3904, Package_TO_SOT_THT:TO-92_Inline, symbol Transistor_BJT:2N3904
- removed U2: ASSR-1218, Package_SO:SO-4_4.4x4.3mm_P2.54mm, symbol Relay_SolidState:ASSR-1218
- added D1: IR26-21C_L110_TR8, LED_SMD:LED_1206_3216Metric, symbol LED:IR26-21C_L110_TR8
- added Q1: MMBT3904, Package_TO_SOT_SMD:SOT-23, symbol Transistor_BJT:MMBT3904
- added R1, R2: 1k, Resistor_SMD:R_1206_3216Metric_Pad1.30x1.75mm_HandSolder, symbol Device:R
Connections:
- net +5V: now also R2.1
- net GND: now also Q1.2 (E)
- net at U1.15 (B0): now also R1.1
- new net: Q1.1 (B), R1.2
- new net: D1.2 (A), R2.2
- no-connect marks 27 -> 25
