File: projects/HA_OPTO_COUPLER_02/HA_OPTO_COUPLER_02.kicad_pcb (KiCad board)
At the start: 0 parts

Commit message: snapshot after creating gerber files for HA_OPTO_COUPLER_02
Parts:
- added J1: TerminalBlock_3pin, UH_HA:Term_Block_1x2_P5mm, F.Cu at (138.4, 94.6)
- added J2: TerminalBlock_3pin, UH_HA:Term_Block_1x2_P5mm, F.Cu at (138.4, 105.4)
- added J3: TerminalBlock_3pin, UH_HA:Term_Block_1x2_P5mm, F.Cu at (162.6, 110.5)
- added J4: TerminalBlock_3pin, UH_HA:Term_Block_1x2_P5mm, F.Cu at (162.6, 99.7)
- added JP1: SolderJumper_3_Open, UH_HA:SolderJumper-3_P2.0mm_Open_TrianglePad1.0x1.5mm_NumberLabels, B.Cu at (153.0, 106.8)
- added JP2: SolderJumper_3_Open, UH_HA:SolderJumper-3_P2.0mm_Open_TrianglePad1.0x1.5mm_NumberLabels, F.Cu at (151.8, 99.1)
- added JP3: SolderJumper_3_Open, UH_HA:SolderJumper-3_P2.0mm_Open_TrianglePad1.0x1.5mm_NumberLabels, B.Cu at (156.2, 106.7)
- added JP4: SolderJumper_3_Open, UH_HA:SolderJumper-3_P2.0mm_Open_TrianglePad1.0x1.5mm_NumberLabels, F.Cu at (151.8, 93.3)
- added Q1: MMBT3904, UH_HA:SOT-23, B.Cu at (149.2, 104.8)
- added Q2: MMBT3904, UH_HA:SOT-23, B.Cu at (149.2, 109.9)
- added R1: 15k, Resistor_SMD:R_0805_2012Metric_Pad1.20x1.40mm_HandSolder, B.Cu at (144.8, 105.4)
- added R2: 200, Resistor_SMD:R_0805_2012Metric_Pad1.20x1.40mm_HandSolder, F.Cu at (144.1, 100.3)
- added R3: 15k, Resistor_SMD:R_0805_2012Metric_Pad1.20x1.40mm_HandSolder, B.Cu at (144.8, 110.5)
- added R4: 200, Resistor_SMD:R_0805_2012Metric_Pad1.20x1.40mm_HandSolder, F.Cu at (144.1, 94.0)
- added T1: HA-OPTO_COUPLER_02, UH_HA:PCB_Name, F.Cu at (150.5, 109.9)
- added T2: (C)UweHerting, UH_HA:Copyright-Uwe_Herting, F.Cu at (149.9, 113.0)
- added T3: https://github.com/uherting/MyKiCADRep, UH_HA:GithubLink_UH, F.Cu at (150.5, 113.7)
- added T4: v0.992, UH_HA:PCB_Version, F.Cu at (149.9, 111.8)
- added U1: EL817, UH_HA:EL817-S1T, B.Cu at (151.8, 100.3)
- added U2: EL817, UH_HA:EL817-S1T, B.Cu at (151.8, 94.6)
Routing:
- net Net-(JP4-Pad1): track 0.00 -> 21.0 mm, vias 0 -> 1
- net Net-(J3-Pad2): track 0.00 -> 14.1 mm
- net Net-(J4-Pad2): track 0.00 -> 13.1 mm
- net Net-(J3-Pad1): track 0.00 -> 12.1 mm
- net Net-(JP3-Pad3): track 0.00 -> 9.86 mm
- net Net-(J4-Pad1): track 0.00 -> 9.66 mm
- net Net-(JP2-Pad1): track 0.00 -> 9.30 mm, vias 0 -> 1
- net Net-(JP4-Pad3): track 0.00 -> 5.52 mm, vias 0 -> 1
- net Net-(JP2-Pad3): track 0.00 -> 5.52 mm, vias 0 -> 1
- net GPIO_2: track 0.00 -> 5.40 mm
- net GPIO_1: track 0.00 -> 5.37 mm
- net Net-(R2-Pad1): track 0.00 -> 5.00 mm, vias 0 -> 1
- net Net-(R4-Pad1): track 0.00 -> 4.73 mm, vias 0 -> 1
- net Net-(JP1-Pad3): track 0.00 -> 4.72 mm
- net Net-(Q2-Pad1): track 0.00 -> 2.64 mm
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- added copper zone on B.Cu, net GND
- added copper zone on F.Cu, net VCC
Other:
- board outline added: 34.3 x 23.5 mm
- copper layers 0 -> 2
