File: projects/HA_OPTO_COUPLER_02/HA_OPTO_COUPLER_02.kicad_sch (KiCad schematic)
At the start: 0 parts

Commit message: snapshot after creating gerber files for HA_OPTO_COUPLER_02
Parts:
- added J1, J2, J3, J4: TerminalBlock_3pin, UH_HA:Term_Block_1x2_P5mm, symbol UH_HA:TerminalBlock_2pin
- added JP1, JP2, JP3, JP4: SolderJumper_3_Open, UH_HA:SolderJumper-3_P2.0mm_Open_TrianglePad1.0x1.5mm_NumberLabels, symbol UH_HA:SolderJumper_3_Open
- added Q1, Q2: MMBT3904, UH_HA:SOT-23, symbol UH_HA:MMBT3904
- added R1, R3: 15k, Resistor_SMD:R_0805_2012Metric_Pad1.20x1.40mm_HandSolder, symbol UH_HA:R
- added R2, R4: 200, Resistor_SMD:R_0805_2012Metric_Pad1.20x1.40mm_HandSolder, symbol UH_HA:R
- added T1: HA-OPTO_COUPLER_02, UH_HA:PCB_Name, symbol UH_HA:PCB_Name
- added T2: (C)UweHerting, UH_HA:Copyright-Uwe_Herting, symbol UH_HA:(C)UweHerting
- added T3: https://github.com/uherting/MyKiCADRep, UH_HA:GithubLink_UH, symbol UH_HA:GithubLink_UH
- added T4: v0.992, UH_HA:PCB_Version, symbol UH_HA:PCB_Version
- added U1, U2: EL817, UH_HA:EL817-S1T, symbol UH_HA:EL817
Connections:
- new net: Q2.1 (B), R3.2
- new net: JP4.1 (A), Q2.3 (C), U2.2
- new net: Q1.1 (B), R1.2
- new net: J4.1, JP3.2 (C)
- new net: JP3.3 (B), U2.4
- new net: R4.1, U2.1
- new net: JP4.3 (B), U2.3
- new net: J3.1, JP1.2 (C)
- new net: JP1.3 (B), U1.4
- new net: R2.1, U1.1
- new net: JP2.1 (A), Q1.3 (C), U1.2
- new net: JP2.3 (B), U1.3
- new net: J3.2, JP2.2 (C)
- new net: J4.2, JP4.2 (C)
- new net +5V: J1.1, R2.2, R4.2
- new net GND: J1.2, JP1.1 (A), JP3.1 (A), Q1.2 (E), Q2.2 (E)
- new net GPIO_1: J2.1, R1.1
- new net GPIO_2: J2.2, R3.1
Other:
- title: (none) -> HA_OPTO_COUPLER_02
