File: projects/HA_OPTO_COUPLER_03/HA_OPTO_COUPLER_03.kicad_pcb (KiCad board)
At the start: 2 copper layers, 34.9 x 34.3 mm, 27 parts, among them J1 TerminalBlock_2pin, J2 TerminalBlock_3pin, J3 TerminalBlock_2pin, J4 TerminalBlock_2pin, J5 TerminalBlock_2pin, Q1 MMBT3904, Q2 MMBT3904, Q3 MMBT3904, T1 HA-OPTO_COUPLER_03, T2 (C)UweHerting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

Commit message: added location for JLCPCB ref num and minor cleanup
Parts:
- added T3: JLCJLCJLCJLC, UH_HA:GithubLink_UH, F.Cu at (153.0, 116.8)
- moved T1 8.26 mm to (154.3, 103.5)
- moved T4 8.26 mm to (154.3, 105.4)
- moved T2 8.25 mm to (154.3, 107.3)
Changed lines of the file:
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@@
       (drillshape 0)
       (scaleselection 1)
-      (outputdirectory "HA_OPTO_COUPLER_03-plots/")
+      (outputdirectory "plots/")
     )
   )
@@
   (net 26 "GPIO_3")
   (footprint "UH_HA:Copyright-Uwe_Herting" (layer "F.Cu")
-    (at 154.305 115.57)
+    (at 154.305 107.315)
     (property "Sheetfile" "HA_OPTO_COUPLER_03.kicad_sch")
     (property "Sheetname" "")
@@
     (fp_line (start -1 0.625) (end -1 -0.625) (layer "F.Fab") (width 0.1))
     (pad "1" smd roundrect (at -1 0 90) (locked) (size 1.2 1.4) (layers "F.Cu" "F.Paste" "F.Mask") (roundrect_rratio 0.2083333333)
-      (net 23 "Net-(R2-Pad1)") (pintype "passive"))
+      (net 23 "Net-(R2-Pad1)"))
     (pad "2" smd roundrect (at 1 0 90) (locked) (size 1.2 1.4) (layers "F.Cu" "F.Paste" "F.Mask") (roundrect_rratio 0.2083333333)
-      (net 9 "VCC") (pintype "passive"))
+      (net 9 "VCC"))
     (model "${KICAD6_3DMODEL_DIR}/Resistor_SMD.3dshapes/R_0805_2012Metric.wrl"
       (offset (xyz 0 0 0))
@@
   )
   (footprint "UH_HA:PCB_Version" (layer "F.Cu")
-    (at 154.305 113.665)
+    (at 154.305 105.41)
     (property "Sheetfile" "HA_OPTO_COUPLER_03.kicad_sch")
     (property "Sheetname" "")
@@
       (rotate (xyz 0 0 0))
     )
+  )
+  (footprint "UH_HA:GithubLink_UH" (layer "F.Cu")
+    (at 153.035 116.84)
+    (property "Sheetfile" "HA_OPTO_COUPLER_03.kicad_sch")
+    (property "Sheetname" "")
+    (fp_text reference "T3" (at 0 1.27 unlocked) (layer "F.Fab") hide
+      (effects (font (size 1 1) (thickness 0.15)))
+    )
+    (fp_text value "JLCJLCJLCJLC" (at 0 -1.27 unlocked) (layer "F.SilkS")
+      (effects (font (size 1 1) (thickness 0.15)))
+    )
+    (fp_line (start -2.54 0) (end 2.54 0) (layer "F.Fab") (width 0.12))
   )
   (footprint "UH_HA:Term_Block_1x2_P5mm" (layer "F.Cu")
@@
   )
   (footprint "UH_HA:PCB_Name" (layer "F.Cu")
-    (at 154.305 111.76)
-    (property "Sheetfile" "HA_OPTO_COUPLER_03.kicad_sch")
-    (property "Sheetname" "")
+    (at 154.305 103.505)
+    (property "Sheetfile" "HA_OPTO_COUPLER_03.kicad_sch")
+    (property "Sheetname" "")
