File: projects/HA_OPTO_COUPLER_03/HA_OPTO_COUPLER_03.kicad_pcb (KiCad board)
At the start: 2 copper layers, 34.9 x 34.3 mm, 28 parts, among them J1 TerminalBlock_2pin, J2 TerminalBlock_3pin, J3 TerminalBlock_2pin, J4 TerminalBlock_2pin, J5 TerminalBlock_2pin, Q1 MMBT3904, Q2 MMBT3904, Q3 MMBT3904, T1 HA-OPTO_COUPLER_03, T2 (C)UweHerting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

Commit message: snapshot after cleaning HA_OPTO_COUPLER_03 project
Parts:
- removed the T3 at (153.0, 116.8)
- removed the T3 at (154.3, 116.8)
- added T3: github.com/uherting/MyKiCADRep, UH_HA:GithubLink_UH, F.Cu at (151.1, 114.3)
- R1, R3, R5: value R -> 15k
- R2, R4, R6: value R -> 200
- T4: value v0.992 -> v0.994
