File: projects/HA_ESP8266_01/HA_ESP8266_01.kicad_pcb (KiCad board)
At the start: 2 copper layers, 45.1 x 67.3 mm, 16 parts, among them J1 IRQs, J2 DataPort A, J3 DataPort B, J4 5V ext, J5 ~RESET, J6 I2C breakout, J7 D5-8 breakout, T1 HA-ESP8266-01, T2 (C)UweHerting, T3 https://github.com/uherting/M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

Commit message: redesigned PCB
Parts:
- added T4: v0.992, UH_HA:PCB_Version, F.Cu at (137.2, 113.0)
- moved U4 5.72 mm to (121.3, 71.1), turned to 90 degrees
- moved J1 4.44 mm to (149.2, 71.1), turned to -90 degrees
- moved T1 3.81 mm to (127.0, 113.0)
- moved J2 2.54 mm to (156.2, 82.5)
- moved U3 1.70 mm to (138.4, 88.9)
- moved U5 1.42 mm to (122.6, 77.5)
- moved J4 1.27 mm to (156.2, 71.1)
- moved U2 0.63 mm to (139.7, 71.1)
Connections:
- J2 pad 10: 3V3 -> 5V
- J2 pad 11: 3V3 -> 5V
- J2 pad 12: 3V3 -> 5V
- J2 pad 13: 3V3 -> 5V
- J2 pad 14: 3V3 -> 5V
- J2 pad 15: 3V3 -> 5V
- J2 pad 16: 3V3 -> 5V
- J2 pad 9: 3V3 -> 5V
- J3 pad 10: 3V3 -> 5V
- J3 pad 11: 3V3 -> 5V
- J3 pad 12: 3V3 -> 5V
- J3 pad 13: 3V3 -> 5V
- J3 pad 14: 3V3 -> 5V
- J3 pad 15: 3V3 -> 5V
- J3 pad 16: 3V3 -> 5V
- J3 pad 9: 3V3 -> 5V
- J6 pad 3: SDA -> SCL
- J6 pad 4: SCL -> SDA
- U1 pad 12: SDA -> SCL
- U1 pad 13: SCL -> SDA
- U3 pad 1: Net-(U2-Pad2) -> Net-(U2-Pad6)
- U3 pad 11: GND -> 3V3
- U3 pad 12: 3V3 -> GND
- U3 pad 13: Net-(J1-Pad2) -> Net-(J1-Pad3)
- U3 pad 14: Net-(J1-Pad3) -> Net-(J1-Pad2)
- U3 pad 3: Net-(U2-Pad6) -> Net-(U2-Pad2)
- U4 pad 1: 3V3 -> GND
- U4 pad 3: GND -> 3V3
Routing:
- net 5V: track 60.8 -> 122.9 mm
- net 3V3: track 154.0 -> 115.6 mm
- net Net-(U2-Pad6): track 12.8 -> 5.39 mm
- net 1WireData3V3: track 47.5 -> 54.8 mm
- net SDA: track 39.7 -> 45.8 mm
- net GND: track 35.6 -> 39.4 mm
- net ~RST: track 8.87 -> 6.88 mm
- net Net-(J3-Pad4): track 20.2 -> 22.1 mm
- net Net-(J3-Pad8): track 20.2 -> 21.9 mm
- net Net-(J3-Pad6): track 20.2 -> 21.9 mm
- net Net-(J3-Pad5): track 20.2 -> 21.9 mm
- net Net-(J3-Pad3): track 20.2 -> 21.9 mm
- net Net-(J3-Pad7): track 20.2 -> 21.9 mm
- net Net-(J3-Pad2): track 20.2 -> 21.9 mm
- net SCL: track 41.4 -> 39.7 mm
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Other:
- board size 45.1 x 67.3 mm -> 46.4 x 67.3 mm

Commit message: updated schema and PCB
Parts:
- LOGO1: moved to B.Cu
- U5: value DS18B20 -> 1WireBus; footprint Package_TO_SOT_THT:TO-92_Inline -> UH_HA:1WireBus
- moved U5 2.62 mm to (120.0, 76.8), turned to 90 degrees
- moved LOGO1 1.65 mm to (130.8, 118.5), turned to 180 degrees
- moved U4 1.27 mm to (120.0, 71.1)
Routing:
- net 1WireData3V3: track 54.8 -> 52.7 mm
- net SDA: track 45.8 -> 45.1 mm
- net GND: vias 0 -> 10

Commit message: snapshot
Other:
- net class Default removed

Commit message: snapshot
Parts:
- removed LOGO1: Logo_Open_Hardware_Small, UH_Symbol:OSHW-Logo2_9.8x8mm_SilkScreen
- added T5: JLCJLCJLCJLC, UH_HA:JLCJLCJLCJLC, F.Cu at (84.5, 149.9)
- J4: value 5V ext -> PWR ext; footprint Connector_PinHeader_2.54mm:PinHeader_1x02_P2.54mm_Vertical -> UH_HA:Term_Block_1x2_P5mm
- T4: value v0.992 -> v0.993
- U2: value I2C addr sel -> I2C addr
- moved J4 47.2 mm to (121.9, 103.5), turned to 0 degrees
- moved J2 44.9 mm to (123.8, 113.7)
- moved J6 44.9 mm to (116.2, 144.1)
- moved T1 44.9 mm to (94.6, 144.1)
- moved T2 44.9 mm to (98.4, 154.3)
- moved U5 44.9 mm to (87.6, 108.0)
- moved T4 44.9 mm to (104.8, 144.1)
- moved U1 44.9 mm to (125.1, 150.5)
- moved J1 44.9 mm to (116.8, 102.2)
- moved J3 44.9 mm to (90.2, 131.4)
- moved J5 44.9 mm to (116.2, 155.6)
- moved J7 44.9 mm to (102.2, 135.3)
- moved T3 44.9 mm to (98.4, 156.8)
- moved U2 44.9 mm to (107.3, 102.2)
- moved U3 44.9 mm to (106.0, 120.0)
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Connections:
- U1 pad 14: Net-(U1-Pad14) -> (no net)
- U1 pad 15: Net-(U1-Pad15) -> (no net)
- U1 pad 19: Net-(U1-Pad19) -> (no net)
- U1 pad 22: Net-(U1-Pad22) -> (no net)
- U1 pad 23: Net-(U1-Pad23) -> (no net)
- U1 pad 24: Net-(U1-Pad24) -> (no net)
- U1 pad 25: Net-(U1-Pad25) -> (no net)
- U1 pad 26: Net-(U1-Pad26) -> (no net)
- U1 pad 27: Net-(U1-Pad27) -> (no net)
- U1 pad 28: Net-(U1-Pad28) -> (no net)
- U1 pad 29: Net-(U1-Pad29) -> (no net)
- U1 pad 3: Net-(U1-Pad3) -> (no net)
- U1 pad 30: Net-(U1-Pad30) -> (no net)
- U1 pad 4: Net-(U1-Pad4) -> (no net)
- U3 pad 4: Net-(U3-Pad4) -> (no net)
- U3 pad 5: Net-(U3-Pad5) -> (no net)
- U3 pad 6: Net-(U3-Pad6) -> (no net)
Routing:
- net 5V: track 122.9 -> 147.3 mm
- net Net-(U2-Pad4): track 9.72 -> 8.98 mm
- net GND: vias 10 -> 11
Other:
- board size 46.4 x 67.3 mm -> 47 x 67.3 mm
