File: projects/HA_ESP8266_01/HA_ESP8266_01.kicad_pcb (KiCad board)
At the start: 2 copper layers, 47 x 67.3 mm, 17 parts, among them J1 IRQs, J2 DataPort A, J3 DataPort B, J4 PWR ext, J5 ~RESET, J6 I2C breakout, J7 D5-8 breakout, T1 HA-ESP8266-01, T2 (C)UweHerting, T3 https://github.com/uherting/M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

Commit message: snapshot prior to changing HA_ESP8266_01 (removing 3pin for one IO and adding 4k7 for dallas 18b20 sensor)
Parts:
- T3: value https://github.com/uherting/MyKiCADRep -> https___github.com_uherting_MyKiCADRep
Connections:
- net ~RST renamed ~{RST}
- U1 pad 14: (no net) -> unconnected-(U1-Pad14)
- U1 pad 15: (no net) -> unconnected-(U1-Pad15)
- U1 pad 19: (no net) -> unconnected-(U1-Pad19)
- U1 pad 22: (no net) -> unconnected-(U1-Pad22)
- U1 pad 23: (no net) -> unconnected-(U1-Pad23)
- U1 pad 24: (no net) -> unconnected-(U1-Pad24)
- U1 pad 25: (no net) -> unconnected-(U1-Pad25)
- U1 pad 26: (no net) -> unconnected-(U1-Pad26)
- U1 pad 27: (no net) -> unconnected-(U1-Pad27)
- U1 pad 28: (no net) -> unconnected-(U1-Pad28)
- U1 pad 29: (no net) -> unconnected-(U1-Pad29)
- U1 pad 3: (no net) -> unconnected-(U1-Pad3)
- U1 pad 30: (no net) -> unconnected-(U1-Pad30)
- U1 pad 4: (no net) -> unconnected-(U1-Pad4)
- U3 pad 4: (no net) -> unconnected-(U3-Pad4)
- U3 pad 5: (no net) -> unconnected-(U3-Pad5)
- U3 pad 6: (no net) -> unconnected-(U3-Pad6)
Changed lines of the file:
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@@
-(kicad_pcb (version 20210228) (generator pcbnew)
+(kicad_pcb (version 20210925) (generator pcbnew)
   (general
     (thickness 1.6)
@@
   (net 13 "Net-(U2-Pad4)")
   (net 14 "Net-(U2-Pad2)")
-  (net 15 "~RST")
+  (net 15 "~{RST}")
   (net 16 "D8")
   (net 17 "Net-(J2-Pad8)")
@@
   (net 31 "Net-(J3-Pad2)")
   (net 32 "Net-(J3-Pad1)")
+  (net 33 "unconnected-(U1-Pad3)")
+  (net 34 "unconnected-(U1-Pad4)")
+  (net 35 "unconnected-(U1-Pad14)")
+  (net 36 "unconnected-(U1-Pad15)")
+  (net 37 "unconnected-(U1-Pad19)")
+  (net 38 "unconnected-(U1-Pad22)")
+  (net 39 "unconnected-(U1-Pad23)")
+  (net 40 "unconnected-(U1-Pad24)")
+  (net 41 "unconnected-(U1-Pad25)")
+  (net 42 "unconnected-(U1-Pad26)")
+  (net 43 "unconnected-(U1-Pad27)")
+  (net 44 "unconnected-(U1-Pad28)")
+  (net 45 "unconnected-(U1-Pad29)")
+  (net 46 "unconnected-(U1-Pad30)")
+  (net 47 "unconnected-(U3-Pad4)")
+  (net 48 "unconnected-(U3-Pad5)")
+  (net 49 "unconnected-(U3-Pad6)")
   (footprint "Connector_PinHeader_2.54mm:PinHeader_1x03_P2.54mm_Vertical" (layer "F.Cu")
     (at 116.84 102.235 -90)
@@
       (net 1 "GND") (pinfunction "Pin_1") (pintype "passive"))
     (pad "2" thru_hole oval locked (at 0 2.54) (size 1.7 1.7) (drill 1) (layers *.Cu *.Mask)
-      (net 15 "~RST") (pinfunction "Pin_2") (pintype "passive"))
+      (net 15 "~{RST}") (pinfunction "Pin_2") (pintype "passive"))
     (model "${KICAD6_3DMODEL_DIR}/Connector_PinHeader_2.54mm.3dshapes/PinHeader_1x02_P2.54mm_Horizontal.wrl"
       (offset (xyz 0 0 0))
@@
       (net 1 "GND") (pinfunction "GND") (pintype "passive"))
     (pad "3" thru_hole oval locked (at -11.43 5.08 270) (size 1.7 1.7) (drill 1) (layers *.Cu *.Mask)
-      (pinfunction "TX") (pintype "bidirectional+no_connect"))
+      (net 33 "unconnected-(U1-Pad3)") (pinfunction "TX") (pintype "bidirectional+no_connect"))
     (pad "4" thru_hole oval locked (at -11.43 7.62 270) (size 1.7 1.7) (drill 1) (layers *.Cu *.Mask)
-      (pinfunction "RX") (pintype "bidirectional+no_connect"))
+      (net 34 "unconnected-(U1-Pad4)") (pinfunction "RX") (pintype "bidirectional+no_connect"))
     (pad "5" thru_hole oval locked (at -11.43 10.16 270) (size 1.7 1.7) (drill 1) (layers *.Cu *.Mask)
       (net 16 "D8") (pinfunction "D8") (pintype "bidirectional"))
@@
       (net 4 "SDA") (pinfunction "D2") (pintype "bidirectional"))
     (pad "14" thru_hole oval locked (at -11.43 33.02 270) (size 1.7 1.7) (drill 1) (layers *.Cu *.Mask)
-      (pinfunction "D1") (pintype "bidirectional+no_connect"))
+      (net 35 "unconnected-(U1-Pad14)") (pinfunction "D1") (pintype "bidirectional+no_connect"))
     (pad "15" thru_hole oval locked (at -11.43 35.56 270) (size 1.7 1.7) (drill 1) (layers *.Cu *.Mask)
-      (pinfunction "D0") (pintype "bidirectional+no_connect"))
+      (net 36 "unconnected-(U1-Pad15)") (pinfunction "D0") (pintype "bidirectional+no_connect"))
     (pad "16" thru_hole circle locked (at 11.43 0 270) (size 1.7 1.7) (drill 1) (layers *.Cu *.Mask)
       (net 3 "5V") (pinfunction "Vin") (pintype "power_in"))
@@
       (net 1 "GND") (pinfunction "GND") (pintype "passive"))
     (pad "18" thru_hole oval locked (at 11.43 5.08 270) (size 1.7 1.7) (drill 1) (layers *.Cu *.Mask)
-      (net 15 "~RST") (pinfunction "~RST") (pintype "power_in"))
+      (net 15 "~{RST}") (pinfunction "~{RST}") (pintype "power_in"))
     (pad "19" thru_hole oval locked (at 11.43 7.62 270) (size 1.7 1.7) (drill 1) (layers *.Cu *.Mask)
-      (pinfunction "EN") (pintype "power_in+no_connect"))
+      (net 37 "unconnected-(U1-Pad19)") (pinfunction "EN") (pintype "power_in+no_connect"))
     (pad "20" thru_hole oval locked (at 11.43 10.16 270) (size 1.7 1.7) (drill 1) (layers *.Cu *.Mask)
       (net 2 "3V3") (pinfunction "3V3") (pintype "passive"))
@@
       (net 1 "GND") (pinfunction "GND") (pintype "passive"))
     (pad "22" thru_hole oval locked (at 11.43 15.24 270) (size 1.7 1.7) (drill 1) (layers *.Cu *.Mask)
-      (pinfunction "CLK") (pintype "no_connect"))
+      (net 38 "unconnected-(U1-Pad22)") (pinfunction "CLK") (pintype "no_connect"))
     (pad "23" thru_hole oval locked (at 11.43 17.78 270) (size 1.7 1.7) (drill 1) (layers *.Cu *.Mask)
-      (pinfunction "SD0") (pintype "no_connect"))
+      (net 39 "unconnected-(U1-Pad23)") (pinfunction "SD0") (pintype "no_connect"))
     (pad "24" thru_hole oval locked (at 11.43 20.32 270) (size 1.7 1.7) (drill 1) (layers *.Cu *.Mask)
-      (pinfunction "CMD") (pintype "no_connect"))
+      (net 40 "unconnected-(U1-Pad24)") (pinfunction "CMD") (pintype "no_connect"))
     (pad "25" thru_hole oval locked (at 11.43 22.86 270) (size 1.7 1.7) (drill 1) (layers *.Cu *.Mask)
-      (pinfunction "SD1") (pintype "no_connect"))
+      (net 41 "unconnected-(U1-Pad25)") (pinfunction "SD1") (pintype "no_connect"))
     (pad "26" thru_hole oval locked (at 11.43 25.4 270) (size 1.7 1.7) (drill 1) (layers *.Cu *.Mask)
-      (pinfunction "SD2") (pintype "no_connect"))
+      (net 42 "unconnected-(U1-Pad26)") (pinfunction "SD2") (pintype "no_connect"))
     (pad "27" thru_hole oval locked (at 11.43 27.94 270) (size 1.7 1.7) (drill 1) (layers *.Cu *.Mask)
-      (pinfunction "SD3") (pintype "no_connect"))
+      (net 43 "unconnected-(U1-Pad27)") (pinfunction "SD3") (pintype "no_connect"))
     (pad "28" thru_hole oval locked (at 11.43 30.48 270) (size 1.7 1.7) (drill 1) (layers *.Cu *.Mask)
-      (pinfunction "RSV2") (pintype "no_connect"))
+      (net 44 "unconnected-(U1-Pad28)") (pinfunction "RSV2") (pintype "no_connect"))
     (pad "29" thru_hole oval locked (at 11.43 33.02 270) (size 1.7 1.7) (drill 1) (layers *.Cu *.Mask)
-      (pinfunction "RSV1") (pintype "no_connect"))
+      (net 45 "unconnected-(U1-Pad29)") (pinfunction "RSV1") (pintype "no_connect"))
     (pad "30" thru_hole oval locked (at 11.43 35.56 270) (size 1.7 1.7) (drill 1) (layers *.Cu *.Mask)
-      (pinfunction "A0") (pintype "input+no_connect"))
+      (net 46 "unconnected-(U1-Pad30)") (pinfunction "A0") (pintype "input+no_connect"))
     (model "${KISYS3DMOD}/Connector_PinSocket_2.54mm.3dshapes/PinSocket_1x15_P2.54mm_Vertical.wrl"
       (offset (xyz -11.43 0 0))
@@
       (effects (font (size 1 1) (thickness 0.15)))
     )
-    (fp_text value "D5-8 breakout" (at 2.54 1.905) (layer "F.Fab")
+    (fp_text value "D5-8 breakout" (at 2.54 3.81) (layer "F.Fab")
       (effects (font (size 1 1) (thickness 0.15)))
     )
@@
       (effects (font (size 1 1) (thickness 0.15)))
     )
-    (fp_text value "https://github.com/uherting/MyKiCADRep" (at 0 1.143 unlocked) (layer "B.SilkS")
+    (fp_text value "https___github.com_uherting_MyKiCADRep" (at 0 1.143 unlocked) (layer "B.SilkS")
       (effects (font (size 1 0.8) (thickness 0.13)) (justify mirror))
     )
@@
       (net 14 "Net-(U2-Pad2)") (pinfunction "ADDR0") (pintype "input"))
     (pad "4" thru_hole oval locked (at -7.62 -3.81) (size 1.7 1.7) (drill 1) (layers *.Cu *.Mask)
-      (pinfunction "~RESET") (pintype "input+no_connect"))
+      (net 47 "unconnected-(U3-Pad4)") (pinfunction "~{RESET}") (pintype "input+no_connect"))
     (pad "5" thru_hole oval locked (at -7.62 -1.27) (size 1.7 1.7) (drill 1) (layers *.Cu *.Mask)
-      (pinfunction "NC/SO") (pintype "no_connect"))
+      (net 48 "unconnected-(U3-Pad5)") (pinfunction "NC/SO") (pintype "no_connect"))
     (pad "6" thru_hole oval locked (at -7.62 1.27) (size 1.7 1.7) (drill 1) (layers *.Cu *.Mask)
-      (pinfunction "NC/CS") (pintype "no_connect"))
+      (net 49 "unconnected-(U3-Pad6)") (pinfunction "NC/CS") (pintype "no_connect"))
     (pad "7" thru_hole oval locked (at -7.62 3.81) (size 1.7 1.7) (drill 1) (layers *.Cu *.Mask)
       (net 4 "SDA") (pinfunction "SDA/SI") (pintype "bidirectional"))
@@
       (net 1 "GND") (pinfunction "GND") (pintype "passive"))
     (pad "13" thru_hole oval locked (at 7.62 -8.89) (size 1.7 1.7) (drill 1) (layers *.Cu *.Mask)
-      (net 10 "Net-(J1-Pad3)") (pinfunction "~ITB") (pintype "output"))
+      (net 10 "Net-(J1-Pad3)") (pinfunction "~{ITB}") (pintype "output"))
     (pad "14" thru_hole oval locked (at 10.16 -8.89) (size 1.7 1.7) (drill 1) (layers *.Cu *.Mask)
-      (net 11 "Net-(J1-Pad2)") (pinfunction "~ITA") (pintype "output"))
+      (net 11 "Net-(J1-Pad2)") (pinfunction "~{ITA}") (pintype "output"))
     (pad "15" thru_hole oval locked (at 7.62 -6.35) (size 1.7 1.7) (drill 1) (layers *.Cu *.Mask)
       (net 25 "Net-(J3-Pad8)") (pinfunction "B0") (pintype "bidirectional"))

Commit message: snapshot
Parts:
- added R1: 4k7, UH_HA:R_0805_2012Metric_Pad1.20x1.40mm_HandSolder, B.Cu at (97.2, 101.6)
- added R2: 4k7, UH_HA:R_0805_2012Metric_Pad1.20x1.40mm_HandSolder, F.Cu at (107.3, 153.0)
- added R3: 4k7, UH_HA:R_0805_2012Metric_Pad1.20x1.40mm_HandSolder, F.Cu at (107.3, 146.7)
- J2: value DataPort A -> DataPort; footprint UH_HA:Dataport_WithPower -> UH_HA:PinHeader_1x08_P2.54mm_Vertical
- J3: value DataPort B -> DataPort; footprint UH_HA:Dataport_WithPower -> UH_HA:PinHeader_1x08_P2.54mm_Vertical
- T3: value https___github.com_uherting_MyKiCADRep -> https://github.com_uherting_MyKiCADRep
- T4: value v0.993 -> v1.0
- moved J3 18.0 mm to (92.7, 113.7), turned to 0 degrees
- moved J2 2.54 mm to (121.3, 113.7)
Connections:
- U3 pad 15: Net-(J3-Pad8) -> Net-(J3-Pad1)
- U3 pad 17: Net-(J3-Pad7) -> Net-(J3-Pad2)
- U3 pad 19: Net-(J3-Pad6) -> Net-(J3-Pad3)
- U3 pad 21: Net-(J3-Pad5) -> Net-(J3-Pad4)
- U3 pad 23: Net-(J3-Pad4) -> Net-(J3-Pad5)
- U3 pad 25: Net-(J3-Pad3) -> Net-(J3-Pad6)
- U3 pad 27: Net-(J3-Pad2) -> Net-(J3-Pad7)
- U3 pad 29: Net-(J3-Pad1) -> Net-(J3-Pad8)
Routing:
- net 5V: track 147.3 -> 87.9 mm
- net GND: track 39.4 -> 3.81 mm
- net 3V3: track 115.7 -> 127.5 mm, vias 0 -> 2
- net SCL: track 39.9 -> 43.1 mm
- net SDA: track 45.1 -> 48.3 mm

Commit message: snapshot
Parts:
- removed T5: JLCJLCJLCJLC, UH_HA:JLCJLCJLCJLC
- removed U5: 1WireBus, UH_HA:1WireBus
- added J10: SSR VCC, Connector_PinHeader_2.54mm:PinHeader_1x03_P2.54mm_Vertical, F.Cu at (94.0, 100.3)
- added J8: D5-8 breakout, Connector_PinHeader_2.54mm:PinHeader_1x06_P2.54mm_Vertical, F.Cu at (102.2, 135.3)
- added J9: SSR out, Connector_PinHeader_2.54mm:PinHeader_1x03_P2.54mm_Vertical, F.Cu at (94.0, 103.5)
- added JP1: A2, UH_HA:SolderJumper-2_P1.3mm_Open_TrianglePad1.0x1.5mm, B.Cu at (105.4, 108.6)
- added JP2: A1, UH_HA:SolderJumper-2_P1.3mm_Open_TrianglePad1.0x1.5mm, B.Cu at (105.4, 111.1)
- added JP3: A0, UH_HA:SolderJumper-2_P1.3mm_Open_TrianglePad1.0x1.5mm, B.Cu at (105.4, 113.7)
- added JP4: SolderJumper_3_Open, UH_HA:SolderJumper-3_P2.0mm_Open_TrianglePad1.0x1.5mm_NumberLabels, F.Cu at (109.2, 102.6)
- added Q1: MMBT3904, UH_HA:SOT-23, F.Cu at (92.7, 109.2)
- added Q2: MMBT3904, UH_HA:SOT-23, F.Cu at (88.9, 110.5)
- added Q3: MMBT3904, UH_HA:SOT-23, F.Cu at (87.0, 116.2)
- added R4: 12k, Resistor_SMD:R_0805_2012Metric_Pad1.20x1.40mm_HandSolder, F.Cu at (92.7, 118.7)
- added R5: 4k7, UH_HA:R_0805_2012Metric_Pad1.20x1.40mm_HandSolder, F.Cu at (107.3, 153.0)
- added R6: 4k7, UH_HA:R_0805_2012Metric_Pad1.20x1.40mm_HandSolder, F.Cu at (107.3, 146.7)
- J2: value DataPort -> DataPort A
- J3: value DataPort -> DataPort B
- J4: value PWR ext -> 5V ext
- J5: value ~RESET -> 5V ext; footprint Connector_PinHeader_2.54mm:PinHeader_1x02_P2.54mm_Horizontal -> Connector_PinHeader_2.54mm:PinHeader_1x02_P2.54mm_Vertical
- J6: value I2C breakout -> ~RESET; footprint Connector_PinHeader_2.54mm:PinHeader_1x04_P2.54mm_Horizontal -> Connector_PinHeader_2.54mm:PinHeader_1x02_P2.54mm_Horizontal
- J7: value D5-8 breakout -> I2C breakout; footprint Connector_PinHeader_2.54mm:PinHeader_1x06_P2.54mm_Vertical -> Connector_PinHeader_2.54mm:PinHeader_1x04_P2.54mm_Horizontal
- R2, R3: value 4k7 -> 12k; footprint UH_HA:R_0805_2012Metric_Pad1.20x1.40mm_HandSolder -> Resistor_SMD:R_0805_2012Metric_Pad1.20x1.40mm_HandSolder
- T1, T2: moved to B.Cu
- T3: value https://github.com_uherting_MyKiCADRep -> https___github.com_uherting_MyKiCADRep; moved to B.Cu
- T4: value v1.0 -> v1.1; moved to B.Cu
- U2: value I2C addr -> MCP23017M; footprint UH_HA:I2C_Address_Selection -> UH_HA:Module_MCP23017
- U3: value MCP23017M -> 1WireBus; footprint UH_HA:Module_MCP23017 -> UH_HA:1WireBus
- moved J5 47.1 mm to (127.6, 109.9), turned to -90 degrees
- moved R2 42.0 mm to (92.7, 113.7), turned to 0 degrees
- moved R3 33.8 mm to (92.7, 116.2), turned to 0 degrees
- moved U2 18.0 mm to (109.8, 120.0), turned to 0 degrees
- moved U4 17.6 mm to (105.1, 100.3), turned to -90 degrees
- moved J7 16.6 mm to (116.3, 144.2), turned to 0 degrees
- moved U3 15.2 mm to (105.2, 104.8), turned to -90 degrees
- moved T4 14.2 mm to (92.1, 150.5), turned to 180 degrees
- moved J6 11.4 mm to (116.3, 155.6)
- moved T1 9.92 mm to (102.2, 150.5), turned to 180 degrees
- moved R1 6.81 mm to (103.9, 102.6)
- moved J4 5.16 mm to (127.0, 102.6), turned to 180 degrees
- moved J3 5.08 mm to (97.8, 113.7)
- moved J2 1.91 mm to (123.2, 113.7)
- moved J1 0.51 mm to (117.3, 102.1)
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Connections:
- J1 pad 2: Net-(J1-Pad2) -> Net-(J1-Pin_2)
- J1 pad 3: Net-(J1-Pad3) -> Net-(J1-Pin_3)
- J2 pad 1: Net-(J2-Pad1) -> Net-(J2-P0)
- J2 pad 2: Net-(J2-Pad2) -> Net-(J2-P1)
- J2 pad 3: Net-(J2-Pad3) -> Net-(J2-P2)
- J2 pad 4: Net-(J2-Pad4) -> Net-(J2-P3)
- J2 pad 5: Net-(J2-Pad5) -> Net-(J2-P4)
- J2 pad 6: Net-(J2-Pad6) -> Net-(J2-P5)
- J2 pad 7: Net-(J2-Pad7) -> Net-(J2-P6)
- J2 pad 8: Net-(J2-Pad8) -> Net-(J2-P7)
- J3 pad 1: Net-(J3-Pad1) -> B0
- J3 pad 2: Net-(J3-Pad2) -> B1
- J3 pad 3: Net-(J3-Pad3) -> B2
- J3 pad 4: Net-(J3-Pad4) -> Net-(J3-P3)
- J3 pad 5: Net-(J3-Pad5) -> Net-(J3-P4)
- J3 pad 6: Net-(J3-Pad6) -> Net-(J3-P5)
- J3 pad 7: Net-(J3-Pad7) -> Net-(J3-P6)
- J3 pad 8: Net-(J3-Pad8) -> Net-(J3-P7)
- J5 pad 1: GND -> 5V
- J5 pad 2: ~{RST} -> GND
- J6 pad 1: 3V3 -> GND
- J6 pad 2: GND -> ~{RST}
- J7 pad 3: D5 -> SCL
- J7 pad 4: D6 -> SDA
- R2 pad 1: 3V3 -> Net-(Q1-B)
- R2 pad 2: SDA -> B0
- R3 pad 1: 3V3 -> Net-(Q2-B)
- R3 pad 2: SCL -> B1
- U2 pad 1: GND -> Net-(JP1-B)
- U2 pad 2: Net-(U2-Pad2) -> Net-(JP2-B)
- U2 pad 3: GND -> Net-(JP3-B)
- U2 pad 4: Net-(U2-Pad4) -> unconnected-(U2-~{RESET}-Pad4)
- U2 pad 5: GND -> unconnected-(U2-NC/SO-Pad5)
- U2 pad 6: Net-(U2-Pad6) -> unconnected-(U2-NC/CS-Pad6)
- U3 pad 1: Net-(U2-Pad6) -> 3V3
- U3 pad 2: Net-(U2-Pad4) -> 1WireData3V3
- U3 pad 3: Net-(U2-Pad2) -> GND
- U4 pad 1: GND -> 3V3
- U4 pad 3: 3V3 -> GND
Routing:
- net B2: track 0.00 -> 24.8 mm
- net B0: track 0.00 -> 24.8 mm
- net B1: track 0.00 -> 24.8 mm
- net Net-(J3-Pad5): track 22.1 -> 0.00 mm
- net Net-(J3-Pad8): track 21.9 -> 0.00 mm
- net Net-(J3-Pad7): track 21.9 -> 0.00 mm
- net Net-(J3-Pad6): track 21.9 -> 0.00 mm
- net Net-(J3-Pad4): track 21.9 -> 0.00 mm
- net Net-(J3-Pad2): track 21.9 -> 0.00 mm
- net Net-(J3-Pad3): track 21.9 -> 0.00 mm
- net Net-(J3-Pad1): track 21.9 -> 0.00 mm
- net Net-(J10-Pin_1): track 0.00 -> 21.3 mm
- net Net-(J3-P7): track 0.00 -> 21.3 mm
- net Net-(J3-P5): track 0.00 -> 20.7 mm
- net Net-(J3-P4): track 0.00 -> 20.7 mm
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Other:
- board size 47 x 67.3 mm -> 47 x 67.7 mm
