File: projects/HA_ESP8266_01/HA_ESP8266_01.kicad_sch (KiCad schematic)
At the start: 17 parts, among them J1 IRQs, J2 DataPort A, J3 DataPort B, J4 5V ext, J5 ~RESET, J6 I2C breakout, J7 D5-8 breakout, T1 HA-ESP8266-01, T2 (C)UweHerting, T3 https://github.com/uherting/M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

Commit message: snapshot
Parts:
- removed J4: 5V ext, Connector_PinHeader_2.54mm:PinHeader_1x02_P2.54mm_Vertical, symbol Connector:Conn_01x02_Male
- removed LOGO1: Logo_Open_Hardware_Small, UH_Symbol:OSHW-Logo2_9.8x8mm_SilkScreen, symbol UH_HA:Logo_Open_Hardware_Small
- removed T3: https://github.com/uherting/MyKiCADRep, UH_HA:GithubLink_UH, symbol UH_HA:GithubLink_UH
- added J4: PWR ext, UH_HA:Term_Block_1x2_P5mm, symbol UH_HA:TerminalBlock_2pin
- added T3: https___github.com_uherting_MyKiCADRep, UH_HA:GithubLink_UH, symbol UH_HA:https___github.com_uherting_MyKiCADRep
- added T5: JLCJLCJLCJLC, UH_HA:JLCJLCJLCJLC, symbol UH_HA:JLCJLCJLCJLC
- T4: value v0.992 -> v0.993
- U2: value I2C addr sel -> I2C addr
Connections:
- net 5V: now also J4.1
- net GND: now also J4.2
- no-connect marks 17 -> 7
Other:
- moved on the sheet: J5

Commit message: snapshot
Parts:
- removed J2: DataPort A, UH_HA:Dataport_WithPower, symbol UH_HA:DataPort_WithPower
- removed J3: DataPort B, UH_HA:Dataport_WithPower, symbol UH_HA:DataPort_WithPower
- added J2, J3: DataPort, UH_HA:PinHeader_1x08_P2.54mm_Vertical, symbol UH_HA:DataPort
- added R1, R2, R3: 4k7, UH_HA:R_0805_2012Metric_Pad1.20x1.40mm_HandSolder, symbol UH_HA:R
- T4: value v0.993 -> v1.0
Connections:
- net 1WireData3V3: now also R1.1
- net 3V3: now also R1.2, R2.1, R3.1
- net SCL: now also R3.2
- net SDA: now also R2.2
- net at U3.15 (B0): now also J3.1 (P0)
- net at U3.16 (A0): now also J2.1 (P0)
- net at U3.17 (B1): now also J3.2 (P1)
- net at U3.18 (A1): now also J2.2 (P1)
- net at U3.19 (B2): now also J3.3 (P2)
- net at U3.20 (A2): now also J2.3 (P2)
- net at U3.21 (B3): now also J3.4 (P3)
- net at U3.22 (A3): now also J2.4 (P3)
- net at U3.23 (B4): now also J3.5 (P4)
- net at U3.24 (A4): now also J2.5 (P4)
- net at U3.25 (B5): now also J3.6 (P5)
- net at U3.26 (A5): now also J2.6 (P5)
- net at U3.27 (B6): now also J3.7 (P6)
- net at U3.28 (A6): now also J2.7 (P6)
- net at U3.29 (B7): now also J3.8 (P7)
- net at U3.30 (A7): now also J2.8 (P7)
- net ~RST renamed ~{RST}
Other:
- moved on the sheet: J6, J7, U4, U5

Commit message: snapshot
Parts:
- removed T5: JLCJLCJLCJLC, UH_HA:JLCJLCJLCJLC, symbol UH_HA:JLCJLCJLCJLC
- removed U2: I2C addr, UH_HA:I2C_Address_Selection, symbol UH_HA:I2C_Address_Selection
- added J10: SSR VCC, Connector_PinHeader_2.54mm:PinHeader_1x03_P2.54mm_Vertical, symbol UH_HA:Conn_01x03_Pin
- added J5: 5V ext, Connector_PinHeader_2.54mm:PinHeader_1x02_P2.54mm_Vertical, symbol UH_HA:Conn_01x02_Pin
- added J9: SSR out, Connector_PinHeader_2.54mm:PinHeader_1x03_P2.54mm_Vertical, symbol UH_HA:Conn_01x03_Pin
- added JP1: A2, UH_HA:SolderJumper-2_P1.3mm_Open_TrianglePad1.0x1.5mm, symbol UH_HA:SolderJumper_2_Open
- added JP2: A1, UH_HA:SolderJumper-2_P1.3mm_Open_TrianglePad1.0x1.5mm, symbol UH_HA:SolderJumper_2_Open
- added JP3: A0, UH_HA:SolderJumper-2_P1.3mm_Open_TrianglePad1.0x1.5mm, symbol UH_HA:SolderJumper_2_Open
- added JP4: SolderJumper_3_Open, UH_HA:SolderJumper-3_P2.0mm_Open_TrianglePad1.0x1.5mm_NumberLabels, symbol UH_HA:SolderJumper_3_Open
- added Q1, Q2, Q3: MMBT3904, UH_HA:SOT-23, symbol UH_HA:MMBT3904
- added R1 (x3): 12k, Resistor_SMD:R_0805_2012Metric_Pad1.20x1.40mm_HandSolder, symbol UH_HA:R
- J1: symbol Connector:Conn_01x03_Male -> UH_HA:Conn_01x03_Pin
- J2: value DataPort -> DataPort A
- J3: value DataPort -> DataPort B
- J4: value PWR ext -> 5V ext
- J6: renamed from J5; symbol Connector:Conn_01x02_Male -> UH_HA:Conn_01x02_Pin
- J7: renamed from J6; symbol Connector:Conn_01x04_Male -> UH_HA:Conn_01x04_Pin
- J8: renamed from J7; symbol Connector:Conn_01x06_Male -> UH_HA:Conn_01x06_Male
- T4: value v1.0 -> v1.1
- renumbered R2 to R5, R3 to R6, U3 to U2, U4 to U3, U5 to U4
Connections:
- net 3V3: now also U3.1 (3V3), U4.1 (3V3), JP4.1 (A); no longer U3.3 (GND), U4.3 (GND)
- net 5V: now also J5.1 (Pin_1), JP4.3 (B)
- net GND: now also U3.3 (GND), U4.3 (GND), J5.2 (Pin_2), JP1.1 (A), JP2.1 (A), JP3.1 (A), Q1.2 (E), Q2.2 (E), Q3.2 (E); no longer U3.1 (3V3), U4.1 (3V3)
- net at U2.1 (ADDR2): now also JP1.2 (B)
- net B0: now reaches J3.1 (P0), U2.15 (B0)
- net B0: now also R1.2
- net B1: now reaches J3.2 (P1), U2.17 (B1)
- net B1: now also R1.2
- net B2: now reaches J3.3 (P2), U2.19 (B2)
- net B2: now also R1.2
- net at U2.2 (ADDR1): now also JP2.2 (B)
- net at U2.3 (ADDR0): now also JP3.2 (B)
- new net: J10.1 (Pin_1), J10.2 (Pin_2), J10.3 (Pin_3), JP4.2 (C)
- new net: Q3.1 (B), R1.1
- new net: Q1.1 (B), R1.1
- new net: Q2.1 (B), R1.1
- new net B0_OUT: J9.1 (Pin_1), Q1.3 (C)
- new net B1_OUT: J9.2 (Pin_2), Q2.3 (C)
- new net B2_OUT: J9.3 (Pin_3), Q3.3 (C)
Other:
- moved on the sheet: J4, J6, J7, J8, R1, R5, R6, U3, U4
